File: v0.1/PCBs/DaughterBoard/MiniRectangleDB.kicad_sch (KiCad schematic)
At the start: 15 parts, among them J1 USB C Connector, J4 Conn_01x06, U2 USBLC6-2SC6

Commit message: Added individual production files
Parts:
- C18: LCSC (none) -> C19666
- F1: LCSC (none) -> C70076
- H3, H5, J4: now left out of the parts list
- J4: LCSC (none) -> C160405
- R1: LCSC C25190 -> C22935
- R2, R3: LCSC C25744 -> C23186
- U2: LCSC (none) -> C7519
Changed lines of the file:
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@@
       (effects (font (size 1.27 1.27)) hide)
     )
-    (property "LCSC" "C25744" (at 87.63 55.753 0)
+    (property "LCSC" "C23186" (at 87.63 55.753 0)
       (effects (font (size 1.27 1.27)) hide)
     )
@@
     )
     (property "Datasheet" "https://www.st.com/resource/en/datasheet/usblc6-2.pdf" (at 52.197 88.265 0)
+      (effects (font (size 1.27 1.27)) hide)
+    )
+    (property "LCSC" "C7519" (at 47.117 97.155 0)
       (effects (font (size 1.27 1.27)) hide)
     )
@@
       (effects (font (size 1.27 1.27)) hide)
     )
-    (property "LCSC" "C25744" (at 90.17 55.753 0)
+    (property "LCSC" "C23186" (at 90.17 55.753 0)
       (effects (font (size 1.27 1.27)) hide)
     )
@@
     )
     (property "Datasheet" "https://www.st.com/resource/en/datasheet/usblc6-2.pdf" (at 104.521 84.963 0)
+      (effects (font (size 1.27 1.27)) hide)
+    )
+    (property "LCSC" "C7519" (at 99.441 93.853 0)
       (effects (font (size 1.27 1.27)) hide)
     )
@@
   )
   (symbol (lib_id "Mechanical:MountingHole") (at 169.799 21.844 0) (unit 1)
-    (in_bom yes) (on_board yes) (dnp no)
+    (in_bom no) (on_board yes) (dnp no)
     (property "Reference" "H5" (at 172.847 21.209 0)
       (effects (font (size 1.27 1.27)) (justify left))
@@
   )
   (symbol (lib_id "Mechanical:MountingHole") (at 141.605 21.844 0) (unit 1)
-    (in_bom yes) (on_board yes) (dnp no)
+    (in_bom no) (on_board yes) (dnp no)
     (property "Reference" "H5" (at 144.653 21.209 0)
       (effects (font (size 1.27 1.27)) (justify left))
@@
   )
   (symbol (lib_id "Mechanical:MountingHole") (at 169.799 28.829 0) (unit 1)
-    (in_bom yes) (on_board yes) (dnp no)
+    (in_bom no) (on_board yes) (dnp no)
     (property "Reference" "H5" (at 172.847 28.194 0)
       (effects (font (size 1.27 1.27)) (justify left))
@@
       (effects (font (size 1.27 1.27)) hide)
     )
+    (property "LCSC" "C70076" (at 95.25 55.753 90)
+      (effects (font (size 1.27 1.27)) hide)
+    )
     (pin "1")
     (pin "2")
@@
       (effects (font (size 1.27 1.27)) hide)
     )
+    (property "LCSC" "C19666" (at 26.67 35.052 90)
+      (effects (font (size 1.27 1.27)) hide)
+    )
     (pin "1")
     (pin "2")
@@
       (effects (font (size 1.27 1.27)) hide)
     )
-    (property "LCSC" "C25190" (at 26.67 30.353 0)
+    (property "LCSC" "C22935" (at 26.67 30.353 0)
       (effects (font (size 1.27 1.27)) hide)
     )
@@
   )
   (symbol (lib_id "Mechanical:MountingHole_Pad") (at 29.21 27.813 0) (mirror y) (unit 1)
-    (in_bom yes) (on_board yes) (dnp no)
+    (in_bom no) (on_board yes) (dnp no)
     (property "Reference" "H3" (at 33.655 24.384 0)
       (effects (font (size 1.27 1.27)) (justify left))
@@
       (effects (font (size 1.27 1.27)) hide)
     )
+    (property "LCSC" "C160405" (at 148.59 74.549 0)
+      (effects (font (size 1.27 1.27)) hide)
+    )
     (pin "1")
     (pin "2")
@@
   )
   (symbol (lib_id "Connector_Generic:Conn_01x06") (at 147.193 45.466 0) (unit 1)
-    (in_bom yes) (on_board yes) (dnp no) (fields_autoplaced)
+    (in_bom no) (on_board yes) (dnp no) (fields_autoplaced)
     (property "Reference" "J4" (at 149.479 46.101 0)
       (effects (font (size 1.27 1.27)) (justify left))
