File: v0.1/PCBs/Main Board/MainBoard.kicad_pcb (KiCad board)
At the start: 2 copper layers, 181.9 x 124.5 mm, 47 parts, among them J1 JTAG_TC2030, J2 FFC Connector, J3 JST Connector, J4 DuPont Connector, SW1 Boot, U1 RP2040, U2 W25Q128JVS, U3 XC6206, Y1 12MHz

Commit message: Added individual production files
Parts:
- R8: value 470 -> 10k
Changed lines of the file:
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@@
     (property "Sheetfile" "MainBoard.kicad_sch")
     (property "Sheetname" "")
+    (property "exclude_from_bom" "")
     (property "ki_description" "Mounting Hole without connection")
     (property "ki_keywords" "mounting hole")
-    (attr through_hole)
+    (attr through_hole exclude_from_pos_files exclude_from_bom)
     (fp_text reference "H1" (at 0 0 90) (layer "F.SilkS") hide
         (effects (font (size 1.27 1.27) (thickness 0.15)))
@@
     (property "Sheetfile" "MainBoard.kicad_sch")
     (property "Sheetname" "")
+    (property "exclude_from_bom" "")
     (property "ki_description" "Mounting Hole without connection")
     (property "ki_keywords" "mounting hole")
-    (attr through_hole)
+    (attr through_hole exclude_from_pos_files exclude_from_bom)
     (fp_text reference "H3" (at 0 0 90) (layer "F.SilkS") hide
         (effects (font (size 1.27 1.27) (thickness 0.15)))
@@
     (property "Sheetfile" "MainBoard.kicad_sch")
     (property "Sheetname" "")
-    (property "exclude_from_bom" "")
     (property "ki_description" "Push button switch, generic, two pins")
     (property "ki_keywords" "switch normally-open pushbutton push-button")
-    (attr smd exclude_from_bom)
+    (attr smd)
     (fp_text reference "SW1" (at 0 3.6 90) (layer "B.SilkS") hide
         (effects (font (size 1 1) (thickness 0.15)) (justify mirror))
@@
         (effects (font (size 0.6 0.6) (thickness 0.15)) (justify mirror))
     )
-    (fp_text value "470" (at 0 -1.17) (layer "B.Fab")
+    (fp_text value "10k" (at 0 -1.17) (layer "B.Fab")
         (effects (font (size 1 1) (thickness 0.15)) (justify mirror))
     )
@@
     (at 175.77104 51.385878 -91)
     (descr "Hotswap footprint for Kailh Choc style switches")
+    (property "LCSC" "C5333465")
     (property "Sheetfile" "MainBoard.kicad_sch")
     (property "Sheetname" "")
@@
     (at 67.034311 82.745087 -123.5)
     (descr "Hotswap footprint for Kailh Choc style switches")
+    (property "LCSC" "C5333465")
     (property "Sheetfile" "MainBoard.kicad_sch")
     (property "Sheetname" "")
@@
     (fp_line (start 9.104 -2.775) (end 7.504 -2.775)
       (stroke (width 0.05) (type solid)) (layer "B.CrtYd"))
-    (fp_arc (start 0.299999 -3.624999) (mid 1.577272 -3.167235) (end 2.455444 -2.13293)
+    (fp_arc (start 0.299999 -3.624999) (mid 1.577271 -3.167235) (end 2.455444 -2.13293)
       (stroke (width 0.05) (type solid)) (layer "B.CrtYd"))
     (fp_arc (start 3.4 -1.475) (mid 2.826424 -1.655848) (end 2.460307 -2.13298)
@@
     (at 44.138321 125.542859 -123.5)
     (descr "Hotswap footprint for Kailh Choc style switches")
+    (property "LCSC" "C5333465")
     (property "Sheetfile" "MainBoard.kicad_sch")
     (property "Sheetname" "")
@@
     (fp_line (start 9.104 -2.775) (end 7.504 -2.775)
       (stroke (width 0.05) (type solid)) (layer "B.CrtYd"))
-    (fp_arc (start 0.299999 -3.624999) (mid 1.577272 -3.167235) (end 2.455444 -2.13293)
+    (fp_arc (start 0.299999 -3.624999) (mid 1.577271 -3.167235) (end 2.455444 -2.13293)
       (stroke (width 0.05) (type solid)) (layer "B.CrtYd"))
     (fp_arc (start 3.4 -1.475) (mid 2.826424 -1.655848) (end 2.460307 -2.13298)
@@
     (at 69.027009 57.828907 -123.5)
     (descr "Hotswap footprint for Kailh Choc style switches")
+    (property "LCSC" "C5333465")
     (property "Sheetfile" "MainBoard.kicad_sch")
     (property "Sheetname" "")
@@
     (fp_line (start 9.104 -2.775) (end 7.504 -2.775)
       (stroke (width 0.05) (type solid)) (layer "B.CrtYd"))
-    (fp_arc (start 0.299999 -3.624999) (mid 1.577272 -3.167235) (end 2.455444 -2.13293)
+    (fp_arc (start 0.299999 -3.624999) (mid 1.577271 -3.167235) (end 2.455444 -2.13293)
       (stroke (width 0.05) (type solid)) (layer "B.CrtYd"))
     (fp_arc (start 3.4 -1.475) (mid 2.826424 -1.655848) (end 2.460307 -2.13298)
@@
     (descr "Resistor SMD 0603 (1608 Metric), square (rectangular) end terminal, IPC_7351 nominal, (Body size source: IPC-SM-782 page 72, https://www.pcb-3d.com/wordpress/wp-content/uploads/ipc-sm-782a_amendment_1_and_2.pdf), generated with kicad-footprint-generator")
     (tags "resistor")
-    (property "LCSC" "C23192")
+    (property "LCSC" "C25804")
     (property "Sheetfile" "MainBoard.kicad_sch")
     (property "Sheetname" "")
@@
     (at 152.530098 59.722749 -121.5)
     (descr "Hotswap footprint for Kailh Choc style switches")
+    (property "LCSC" "C5333465")
     (property "Sheetfile" "MainBoard.kicad_sch")
     (property "Sheetname" "")
@@
     (at 89.358451 45.276002 -123.5)
     (descr "Hotswap footprint for Kailh Choc style switches")
+    (property "LCSC" "C5333465")
     (property "Sheetfile" "MainBoard.kicad_sch")
     (property "Sheetname" "")
@@
     (fp_line (start 9.104 -2.775) (end 7.504 -2.775)
       (stroke (width 0.05) (type solid)) (layer "B.CrtYd"))
-    (fp_arc (start 0.299999 -3.624999) (mid 1.577272 -3.167235) (end 2.455444 -2.13293)
+    (fp_arc (start 0.299999 -3.624999) (mid 1.577271 -3.167235) (end 2.455444 -2.13293)
       (stroke (width 0.05) (type solid)) (layer "B.CrtYd"))
     (fp_arc (start 3.4 -1.475) (mid 2.826424 -1.655848) (end 2.460307 -2.13298)
@@
     (property "Sheetfile" "MainBoard.kicad_sch")
     (property "Sheetname" "")
+    (property "exclude_from_bom" "")
     (property "ki_description" "Mounting Hole without connection")
     (property "ki_keywords" "mounting hole")
-    (attr through_hole)
+    (attr through_hole exclude_from_pos_files exclude_from_bom)
     (fp_text reference "H4" (at 0 0 90) (layer "B.SilkS") hide
         (effects (font (size 1.27 1.27) (thickness 0.15)) (justify mirror))
@@
     (at 72.296424 111.713906 -123.5)
     (descr "Hotswap footprint for Kailh Choc style switches")
+    (property "LCSC" "C5333465")
     (property "Sheetfile" "MainBoard.kicad_sch")
     (property "Sheetname" "")
@@
     (fp_line (start 9.104 -2.775) (end 7.504 -2.775)
       (stroke (width 0.05) (type solid)) (layer "B.CrtYd"))
-    (fp_arc (start 0.299999 -3.624999) (mid 1.577272 -3.167235) (end 2.455444 -2.13293)
+    (fp_arc (start 0.299999 -3.624999) (mid 1.577271 -3.167235) (end 2.455444 -2.13293)
       (stroke (width 0.05) (type solid)) (layer "B.CrtYd"))
     (fp_arc (start 3.4 -1.475) (mid 2.826424 -1.655848) (end 2.460307 -2.13298)
@@
     (property "Sheetfile" "MainBoard.kicad_sch")
     (property "Sheetname" "")
+    (property "exclude_from_bom" "")
     (property "ki_description" "Mounting Hole without connection")
     (property "ki_keywords" "mounting hole")
-    (attr through_hole)
+    (attr through_hole exclude_from_pos_files exclude_from_bom)
     (fp_text reference "H2" (at 0 0 90) (layer "B.SilkS") hide
         (effects (font (size 1.27 1.27) (thickness 0.15)) (justify mirror))
@@
     (property "Sheetfile" "MainBoard.kicad_sch")
     (property "Sheetname" "")
+    (property "exclude_from_bom" "")
     (property "ki_description" "6-pin TC2030 connector for JTAG programming")
     (property "ki_keywords" "JTAG ARM SWD connector tag connect tc 2030")
-    (attr exclude_from_pos_files)
+    (attr exclude_from_pos_files exclude_from_bom)
     (fp_text reference "J1" (at 0 -2.7 90) (layer "B.SilkS")
         (effects (font (size 1 1) (thickness 0.15)) (justify mirror))
