File: v0.1/PCBs/Main Board/MainBoard.kicad_sch (KiCad schematic)
At the start: 47 parts, among them J2 DuPont Connector, J2 FFC Connector, J2 JTAG_TC2030, J3 JST Connector, SW1 Boot, U1 XC6206, U3 RP2040, U4 W25Q128JVS, Y1 12MHz

Commit message: Added individual production files
Parts:
- CH1, CH2, CH3, CH4, CH5, CH6, CH7: LCSC (none) -> C5333465
- H1, H2, H3, H4, J2: now left out of the parts list
- R4: value 470 -> 10k
- R6: LCSC C23192 -> C25804
- SW1: now in the parts list
Changed lines of the file:
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@@
+      (effects (font (size 1.27 1.27)) hide)
+    )
+    (property "LCSC" "C5333465" (at 154.178 51.435 0)
       (effects (font (size 1.27 1.27)) hide)
     )
@@
   )
   (symbol (lib_id "Mechanical:MountingHole") (at 203.2 30.988 0) (unit 1)
-    (in_bom yes) (on_board yes) (dnp no)
+    (in_bom no) (on_board yes) (dnp no)
     (property "Reference" "H3" (at 205.74 29.718 0)
       (effects (font (size 1.27 1.27)) (justify left) hide)
@@
     )
     (property "Datasheet" "~" (at 125.095 50.419 0)
+      (effects (font (size 1.27 1.27)) hide)
+    )
+    (property "LCSC" "C5333465" (at 125.095 50.419 0)
       (effects (font (size 1.27 1.27)) hide)
     )
@@
       (effects (font (size 1.27 1.27)) hide)
     )
+    (property "LCSC" "C5333465" (at 139.573 46.609 0)
+      (effects (font (size 1.27 1.27)) hide)
+    )
     (pin "1")
     (pin "2")
@@
       (effects (font (size 1.27 1.27)) hide)
     )
-    (property "LCSC" "C23192" (at 200.5239 157.0501 0)
+    (property "LCSC" "C25804" (at 200.5239 157.0501 0)
       (effects (font (size 1.27 1.27)) hide)
     )
@@
       (effects (font (size 1.27 1.27)) hide)
     )
+    (property "LCSC" "C5333465" (at 161.671 97.79 0)
+      (effects (font (size 1.27 1.27)) hide)
+    )
     (pin "1")
     (pin "2")
@@
     )
     (property "Datasheet" "~" (at 108.331 34.798 0)
+      (effects (font (size 1.27 1.27)) hide)
+    )
+    (property "LCSC" "C5333465" (at 108.331 34.798 0)
       (effects (font (size 1.27 1.27)) hide)
     )
@@
       (effects (font (size 1.27 1.27)) hide)
     )
+    (property "LCSC" "C5333465" (at 168.656 54.737 0)
+      (effects (font (size 1.27 1.27)) hide)
+    )
     (pin "1")
     (pin "2")
@@
   )
   (symbol (lib_id "Mechanical:MountingHole") (at 189.23 35.179 0) (unit 1)
-    (in_bom yes) (on_board yes) (dnp no)
+    (in_bom no) (on_board yes) (dnp no)
     (property "Reference" "H2" (at 191.77 33.909 0)
       (effects (font (size 1.27 1.27)) (justify left) hide)
@@
   )
   (symbol (lib_id "marbastlib-various:JTAG_TC2030") (at 161.798 180.213 0) (unit 1)
-    (in_bom yes) (on_board yes) (dnp no)
+    (in_bom no) (on_board yes) (dnp no)
     (property "Reference" "J2" (at 169.0878 177.6729 0)
       (effects (font (size 1.27 1.27)) (justify left))
@@
       (effects (font (size 1.27 1.27)) (justify left))
     )
-    (property "Value" "470" (at 240.275 156.4486 90)
+    (property "Value" "10k" (at 240.275 156.4486 90)
       (effects (font (size 0.8 0.8)) (justify left))
     )
@@
       (effects (font (size 1.27 1.27)) hide)
     )
+    (property "LCSC" "C5333465" (at 150.622 85.344 0)
+      (effects (font (size 1.27 1.27)) hide)
+    )
     (pin "1")
     (pin "2")
@@
   )
   (symbol (lib_id "Mechanical:MountingHole") (at 203.2 35.179 0) (unit 1)
-    (in_bom yes) (on_board yes) (dnp no)
+    (in_bom no) (on_board yes) (dnp no)
     (property "Reference" "H4" (at 205.74 33.909 0)
       (effects (font (size 1.27 1.27)) (justify left) hide)
@@
   )
   (symbol (lib_id "Mechanical:MountingHole") (at 189.23 30.988 0) (unit 1)
-    (in_bom yes) (on_board yes) (dnp no)
+    (in_bom no) (on_board yes) (dnp no)
     (property "Reference" "H1" (at 191.77 29.718 0)
       (effects (font (size 1.27 1.27)) (justify left) hide)
@@
   )
   (symbol (lib_id "Switch:SW_Push") (at 109.093 134.493 0) (unit 1)
-    (in_bom no) (on_board yes) (dnp no) (fields_autoplaced)
+    (in_bom yes) (on_board yes) (dnp no) (fields_autoplaced)
     (property "Reference" "SW1" (at 109.093 127.6055 0)
       (effects (font (size 1.27 1.27)))
